Commit message: Update: completed rough draft of model chassis
Very basic robot model

File: urdf/eng405_bot.xacro (robot description, xacro)
@@ -7,3 +7,28 @@
 		<child link="chassis"/>
 	</joint>
+	<!--Robot main chassis-->
+	<link name="chassis">
+		<pose>0 0 0.1 0 0 0</pose>
+		<inertial>
+			<mass value="15.0"/>
+			<origin xyz="0 0 0" rpy="0 0 0"/>
+			<inertia
+				ixx="0.1" ixy="0" ixz="0"
+				iyy="0.1" iyz="0"
+				izz="0.1"
+			/>
+		</inertial>
+		<collision name="collision">
+			<origin xyz="0 0 0" rpy="0 0 0"/>
+			<geometry>
+				<box size="0.4 0.2 0.1" />
+			</geometry>
+		</collision>
+		<visual name="chassis_visual">
+			<origin xyz="0 0 0" rpy="0 0 0"/>
+			<geometry>
+				<box size="0.4 0.2 0.1"/>
+			</geometry>
+		</visual>
+	</link>
 </robot>

Commit message: Update: robot model finished
Added the wheel geometries and the camera and LRF geometries - still need to get the model fully working

File: urdf/eng405_bot.xacro (robot description, xacro)
@@ -1,5 +1,7 @@
 <?xml version="1.0"?>
 <robot name="eng405_bot" xmlns:xacro="http://www.ros.org/wiki/xacro">
+	<!-- Robot footprint -->
 	<link name="robot_footprint"></link>
+	<!-- Joint from robot footprint to chassis -->
 	<joint name="robot_footprint_joint" type="fixed">
 		<origin xyz="0 0 0" rpy="0 0 0"/>
@@ -11,5 +13,5 @@
 		<pose>0 0 0.1 0 0 0</pose>
 		<inertial>
-			<mass value="15.0"/>
+			<mass value="1.0"/>
 			<origin xyz="0 0 0" rpy="0 0 0"/>
 			<inertia
@@ -19,16 +21,195 @@
 			/>
 		</inertial>
-		<collision name="collision">
-			<origin xyz="0 0 0" rpy="0 0 0"/>
-			<geometry>
-				<box size="0.4 0.2 0.1" />
-			</geometry>
-		</collision>
-		<visual name="chassis_visual">
-			<origin xyz="0 0 0" rpy="0 0 0"/>
-			<geometry>
-				<box size="0.4 0.2 0.1"/>
-			</geometry>
-		</visual>
-	</link>
+		<!-- main chassis -->
+		<collision name="main_chassis_collision">
+			<origin xyz="0 0 0" rpy="0 0 0"/>
+			<geometry>
+				<box size="0.17 0.09 0.05" />
+			</geometry>
+		</collision>
+		<visual name="main_chassis_visual">
+			<origin xyz="0 0 0" rpy="0 0 0"/>
+			<geometry>
+				<box size="0.17 0.09 0.05"/>
+			</geometry>
+		</visual>
+		<!-- Battery brick -->
+		<collision name="battery_brick_collision">
+			<origin xyz="-0.035 0 0.06" rpy="0 0 0"/>
+			<geometry>
+				<box size="0.1 0.09 0.07"/>
+			</geometry>
+		</collision>
+		<visual name="battery_brick_visual">
+			<origin xyz="-0.035 0 0.06" rpy="0 0 0"/>
+			<geometry>
+				<box size="0.1 0.09 0.07"/>
+			</geometry>
+		</visual>
+		<!-- right chassis -->
+		<collision name="right_chassis_collision">
+			<origin xyz="-0.065 -0.055 0" rpy="0 -0.52359 0"/>
+			<geometry>
+				<box size="0.1 0.02 0.035" />
+			</geometry>
+		</collision>
+		<visual name="right_chassis_visual">
+			<origin xyz="-0.065 -0.055 0" rpy="0 -0.52359 0"/>
+			<geometry>
+				<box size="0.1 0.02 0.035"/>
+			</geometry>
+		</visual>
+		<!-- left chassis -->
+		<collision name="left_chassis_collision">
+			<origin xyz="-0.065 0.055 0" rpy="0 -0.52359 0"/>
+			<geometry>
+				<box size="0.1 0.02 0.035" />
+			</geometry>
+		</collision>
+		<visual name="left_chassis_visual">
+			<origin xyz="-0.065 0.055 0" rpy="0 -0.52359 0"/>
+			<geometry>
+				<box size="0.1 0.02 0.035"/>
+			</geometry>
+		</visual>
+		<!-- Castor at front of robot -->
+		<collision name="front_caster_collision">
+			<origin xyz="0.04 0 -0.025" rpy="0 0 0"/>
+			<geometry>
+				<sphere radius="0.025"/>
+			</geometry>
+		</collision>
+		<visual name="front_caster_visual">
+			<origin xyz="0.04 0 -0.025" rpy="0 0 0"/>
+			<geometry>
+				<sphere radius="0.025"/>
+			</geometry>
+		</visual>
+	</link>
+	<!-- Robot right wheel -->
+	<link name="right_wheel">
+		<inertial>
+			<mass value="0.1"/>
+			<origin xyz="0 0 0" rpy="0 1.5707 1.5707"/>
+			<inertia
+				ixx="0.1" ixy="0" ixz="0"
+				iyy="0.1" iyz="0"
+				izz="0.1"
+			/>
+		</inertial>
+		<collision>
+			<origin xyz="0 0 0" rpy="0 1.5707 1.5707"/>
+			<geometry>
+				<cylinder length="0.005" radius="0.03"/>
+			</geometry>
+		</collision>
+		<visual>
+			<origin xyz="0 0 0" rpy="0 1.5707 1.5707"/>
+			<geometry>
+				<cylinder length="0.005" radius="0.03"/>
+			</geometry>
+		</visual>
+	</link>
+	<!-- Robot left wheel -->
+	<link name="left_wheel">
+		<inertial>
+			<mass value="0.1"/>
+			<origin xyz="0 0 0" rpy="0 1.5707 1.5707"/>
+			<inertia
+				ixx="0.1" ixy="0" ixz="0"
+				iyy="0.1" iyz="0"
+				izz="0.1"
+			/>
+		</inertial>
+		<collision>
+			<origin xyz="0 0 0" rpy="0 1.5707 1.5707"/>
+			<geometry>
+				<cylinder length="0.005" radius="0.03"/>
+			</geometry>
+		</collision>
+		<visual>
+			<origin xyz="0 0 0" rpy="0 1.5707 1.5707"/>
+			<geometry>
+				<cylinder length="0.005" radius="0.03"/>
+			</geometry>
+		</visual>
+	</link>
+	<!-- Joint to connect right wheel to chassis -->
+	<joint type="continuous" name="right_wheel_hinge">
+		<origin xyz="-0.099641 -0.075 -0.02" rpy="0 0 0"/>
+		<child link="right_wheel"/>
+		<parent link="chassis"/>
+		<axis xyz="0 1 0" rpy="0 0 0"/>
+		<limit effort="10000" velocity="1000"/>
+		<dynamics damping="1.0" friction="1.0"/>
+	</joint>
+	<!-- Joint to connect left wheel to chassis -->
+	<joint type="continuous" name="left_wheel_hinge">
+		<origin xyz="-0.099641 0.075 -0.02" rpy="0 0 0"/>
+		<child link="left_wheel"/>
+		<parent link="chassis"/>
+		<axis xyz="0 1 0" rpy="0 0 0"/>
+		<limit effort="10000" velocity="1000"/>
+		<dynamics damping="1.0" friction="1.0"/>
+	</joint>
+	<!-- Camera -->
+	<link name="camera">
+		<inertial>
+			<mass value="0.1"/>
+			<origin xyz="0 0 0" rpy="0 0 0"/>
+			<inertia
+				ixx="1e-6" ixy="0" ixz="0"
+				iyy="1e-6" iyz="0"
+				izz="1e-6"
+			/>
+		</inertial>
+		<collision>
+			<origin xyz="0 0 0" rpy="0 0 0"/>
+			<geometry>
+				<box size="0.025 0.025 0.025"/>
+			</geometry>
+		</collision>
+		<visual>
+			<origin xyz="0 0 0" rpy="0 0 0"/>
+			<geometry>
+				<box size="0.025 0.025 0.025"/>
+			</geometry>
+		</visual>
+	</link>
+	<!-- Joint connecting the camera to the chassis -->
+	<joint type="fixed" name="camera_joint">
+		<origin xyz="0.09 0 0" rpy="0 0 0"/>
+		<parent link="chassis"/>
+		<child link="camera"/>
+	</joint>
+	<!-- Laser Range Finder -->
+	<link name="hokuyo">
+		<inertial>
+			<mass value="0.1"/>
+			<origin xyz="0 0 0" rpy="0 0 0"/>
+			<inertia
+				ixx="1e-6" ixy="0" ixz="0"
+				iyy="1e-6" iyz="0"
+				izz="1e-6"
+			/>
+		</inertial>
+		<collision>
+			<origin xyz="0 0 0" rpy="0 0 0"/>
+			<geometry>
+				<box size="0.1 0.1 0.1"/>
+			</geometry>
+		</collision>
+		<visual>
+			<origin xyx="0 0 0" rpy="0 0 0"/>
+			<geometry>
+				<mesh filename="package://eng405_bot/meshes/hokuyo.dae"/>
+			</geometry>
+		</visual>
+	</link>
+	<!-- Joint connecting the chassis with the LRF -->
+	<joint type="fixed" name="hokuyo_joint">
+		<origin xyz="-0.035 0 0.1" rpy="0 0 0"/>
+		<parent link="chassis"/>
+		<child link="hokuyo"/>
+	</joint>
 </robot>

Commit message: Update: colours to the robot model in Gazebo and also imported the materials xacro to robot model

File: urdf/eng405_bot.xacro (robot description, xacro)
@@ -3,4 +3,6 @@
 	<!-- Gazebo file used to load the plugins for gazebo for DD, camera, and LRF -->
 	<xacro:include filename="$(find eng405_bot)/urdf/eng405_bot.gazebo"/>
+	<!-- Import the Rviz colors -->
+	<xacro:include filename="$(find eng405_bot)/urdf/materials.xacro"/>
 	<!-- Robot footprint -->
 	<link name="robot_footprint"></link>
@@ -35,4 +37,5 @@
 				<box size="0.17 0.09 0.05"/>
 			</geometry>
+			<material name="blue"/>
 		</visual>
 		<!-- Battery brick -->
@@ -48,4 +51,5 @@
 				<box size="0.1 0.09 0.07"/>
 			</geometry>
+			<material name="blue"/>
 		</visual>
 		<!-- right chassis -->
@@ -61,4 +65,5 @@
 				<box size="0.1 0.02 0.035"/>
 			</geometry>
+			<material name="blue"/>
 		</visual>
 		<!-- left chassis -->
@@ -74,4 +79,5 @@
 				<box size="0.1 0.02 0.035"/>
 			</geometry>
+			<material name="blue"/>
 		</visual>
 		<!-- Castor at front of robot -->

Commit message: Update: changed the launch files to accomodate Rviz
Changed the robot model for Rviz colour and amended some errors in the camera plugin

File: urdf/eng405_bot.xacro (robot description, xacro)
@@ -117,4 +117,5 @@
 				<cylinder length="0.005" radius="0.03"/>
 			</geometry>
+			<material name="green"/>
 		</visual>
 	</link>
@@ -141,4 +142,5 @@
 				<cylinder length="0.005" radius="0.03"/>
 			</geometry>
+			<material name="green"/>
 		</visual>
 	</link>
@@ -217,5 +219,5 @@
 	<!-- Joint connecting the chassis with the LRF -->
 	<joint type="fixed" name="hokuyo_joint">
-		<origin xyz="-0.035 0 0.1" rpy="0 0 0"/>
+		<origin xyz="-0.035 0 0.14" rpy="0 0 0"/>
 		<parent link="chassis"/>
 		<child link="hokuyo"/>

Commit message: Update: changed some parameters

File: urdf/eng405_bot.xacro (robot description, xacro)
@@ -17,10 +17,10 @@
 		<pose>0 0 0.1 0 0 0</pose>
 		<inertial>
-			<mass value="1.0"/>
-			<origin xyz="0 0 0" rpy="0 0 0"/>
-			<inertia
-				ixx="0.1" ixy="0" ixz="0"
-				iyy="0.1" iyz="0"
-				izz="0.1"
+			<mass value="3.0"/>
+			<origin xyz="0 0 0" rpy="0 0 0"/>
+			<inertia
+				ixx="0.02" ixy="0" ixz="0"
+				iyy="0.02" iyz="0"
+				izz="0.02"
 			/>
 		</inertial>
@@ -87,4 +87,14 @@
 				<sphere radius="0.025"/>
 			</geometry>
+			<surface>
+        		<friction>
+          			<ode>
+            			<mu>0.0</mu>
+            			<mu2>0.0</mu2>
+            			<slip1>1.0</slip1>
+            			<slip2>1.0</slip2>
+          			</ode>
+        		</friction>
+      		</surface>
 		</collision>
 		<visual name="front_caster_visual">
@@ -98,10 +108,10 @@
 	<link name="right_wheel">
 		<inertial>
-			<mass value="0.1"/>
-			<origin xyz="0 0 0" rpy="0 1.5707 1.5707"/>
-			<inertia
-				ixx="0.1" ixy="0" ixz="0"
-				iyy="0.1" iyz="0"
-				izz="0.1"
+			<mass value="1"/>
+			<origin xyz="0 0 0" rpy="0 1.5707 1.5707"/>
+			<inertia
+				ixx="0.02" ixy="0" ixz="0"
+				iyy="0.02" iyz="0"
+				izz="0.02"
 			/>
 		</inertial>
@@ -123,10 +133,10 @@
 	<link name="left_wheel">
 		<inertial>
-			<mass value="0.1"/>
-			<origin xyz="0 0 0" rpy="0 1.5707 1.5707"/>
-			<inertia
-				ixx="0.1" ixy="0" ixz="0"
-				iyy="0.1" iyz="0"
-				izz="0.1"
+			<mass value="1"/>
+			<origin xyz="0 0 0" rpy="0 1.5707 1.5707"/>
+			<inertia
+				ixx="0.02" ixy="0" ixz="0"
+				iyy="0.02" iyz="0"
+				izz="0.02"
 			/>
 		</inertial>
